File: pcb/soil_sensor_2.kicad_pcb (KiCad board)
At the start: 2 copper layers, 26 x 120.3 mm, 29 parts, among them J1 532610471, J2 ESP-PROG, Q1 SI2312, U1 SHT4x, U2 TPS61201DRCT, U3 ESP32-PICO-V3

Commit message: chore: add cutout to improve temperature isolation
Parts:
- moved C1 1.70 mm to (115.7, 86.5)
- moved U1 1.70 mm to (113.7, 86.5)
Routing:
- net +3V3: track 48.9 -> 51.2 mm
- net /SCL_{0}: track 9.11 -> 11.0 mm
- net /SDA_{0}: track 10.2 -> 12.1 mm
- net GND: vias 182 -> 178
Other:
- outline, holes or cut-outs redrawn
- board text added: "REV 1.3.1 01-05-2022"
- board text removed: "REV 1.3 09-12-2021"
